File: Power_switch.kicad_sch (KiCad schematic)
At the start: 36 parts, among them Q409 AO3400A, Q410 HSBA8119, Q415 MMBT5551, Q416 AO3400A, Q417 HSBA8119, SW401 SW_SPDT, U400 INA219AIDCNR, U407 INA219AIDCNR, U408 INA219AIDCNR

Commit message: generated final gerber
Parts:
- IC408: value ~ -> (none)
