File: mcu.kicad_sch (KiCad schematic)
At the start: 46 parts, among them Q404 AO3400A, U405 STM32H562VGTx, X300 Q13FC1350000400, Y400 ASE-xxxMHz

Commit message: generated final gerber
Parts:
- FB401: value ~ -> (none)
Changed lines of the file:
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@@
 (kicad_sch
-	(version 20250114)
+	(version 20260306)
 	(generator "eeschema")
-	(generator_version "9.0")
+	(generator_version "10.0")
 	(paper "A3")
 	(title_block
